File: 16bit_computer.kicad_sch (KiCad schematic)
At the start: 24 parts, among them J1 Conn_01x03, J2 Conn_01x16_Male, U1 40374, U2 40374, U3 40245, U4 40245, U5 7408

Commit message: register finished?
Parts:
- removed D1, D10, D11, D12, D13, D14, D15, D16, D2, D3, D4, D5, D6, D7, D8, D9: LED, Diode_SMD:D_0603_1608Metric_Pad1.05x0.95mm_HandSolder_BETTER, symbol Device:LED
- removed JA1: Conn_01x02, Connector_PinHeader_2.54mm:PinHeader_1x02_P2.54mm_Vertical, symbol Connector_Generic:Conn_01x02
- removed U1, U2: 40374, Package_DIP:DIP-20_W7.62mm_Socket_LongPads, symbol 4xxx_IEEE:40374
- removed U3, U4: 40245, Package_DIP:DIP-20_W7.62mm_Socket_LongPads, symbol 4xxx_IEEE:40245
- added J7, J8: Conn_01x16, Connector_PinHeader_2.54mm:PinHeader_1x16_P2.54mm_Vertical, symbol Connector_Generic:Conn_01x16
- added REG1, REG2, REG3, REG4: Conn_01x02, Connector_PinHeader_2.54mm:PinHeader_1x02_P2.54mm_Vertical, symbol Connector_Generic:Conn_01x02
Connections:
- net LD_A is gone; now on net CLK: U5.5 (Pin_5)
- net CLK: now also U5.12 (Pin_12), U5.2 (Pin_2), U5.9 (Pin_9); no longer U5.4 (Pin_4)
- net at U5.1 (Pin_1): now also REG3.2 (Pin_2)
- net at U5.10 (Pin_10): now also REG4.2 (Pin_2)
- net Register2/LOAD: now reaches U5.11 (Pin_11)
- net at U5.13 (Pin_13): now also REG2.2 (Pin_2)
- net Register3/LOAD: now reaches U5.3 (Pin_3)
- net Register4/LOAD: now reaches U5.8 (Pin_8)
- net 1 renamed BUS1
- net BUS1: now also J7.1 (Pin_1), J8.1 (Pin_1)
- net 10 renamed BUS10
- net BUS10: now also J7.10 (Pin_10), J8.10 (Pin_10)
- net 11 renamed BUS11
- net BUS11: now also J7.11 (Pin_11), J8.11 (Pin_11)
- net 12 renamed BUS12
- net BUS12: now also J7.12 (Pin_12), J8.12 (Pin_12)
- net 13 renamed BUS13
- net BUS13: now also J7.13 (Pin_13), J8.13 (Pin_13)
- net 14 renamed BUS14
- net BUS14: now also J7.14 (Pin_14), J8.14 (Pin_14)
- net 15 renamed BUS15
- net BUS15: now also J7.15 (Pin_15), J8.15 (Pin_15)
- net 16 renamed BUS16
- net BUS16: now also J7.16 (Pin_16), J8.16 (Pin_16)
- net 2 renamed BUS2
- net BUS2: now also J7.2 (Pin_2), J8.2 (Pin_2)
- net 3 renamed BUS3
- net BUS3: now also J7.3 (Pin_3), J8.3 (Pin_3)
- net 4 renamed BUS4
- net BUS4: now also J7.4 (Pin_4), J8.4 (Pin_4)
- net 5 renamed BUS5
- net BUS5: now also J7.5 (Pin_5), J8.5 (Pin_5)
- net 6 renamed BUS6
- net BUS6: now also J7.6 (Pin_6), J8.6 (Pin_6)
- net 7 renamed BUS7
- net BUS7: now also J7.7 (Pin_7), J8.7 (Pin_7)
- net 8 renamed BUS8
- net BUS8: now also J7.8 (Pin_8), J8.8 (Pin_8)
- net 9 renamed BUS9
- net BUS9: now also J7.9 (Pin_9), J8.9 (Pin_9)
- net LOAD_A renamed Register1/LOAD
- new net: REG1.2 (Pin_2), U5.4 (Pin_4)
- new net Register1/~{ENABLE}: REG1.1 (Pin_1)
- new net Register2/~{ENABLE}: REG2.1 (Pin_1)
- new net Register3/~{ENABLE}: REG3.1 (Pin_1)
- new net Register4/~{ENABLE}: REG4.1 (Pin_1)
Other:
- sheet Register renamed Register1
- added sheet Register2 (register.kicad_sch)
- added sheet Register3 (register.kicad_sch)
- added sheet Register4 (register.kicad_sch)
- sheet Register1 ports: added BUS[1..16], LOAD, ~{ENABLE}; removed none
- moved on the sheet: U5
