File: register.kicad_sch (KiCad schematic)
At the start: 0 parts

Commit message: register finished?
Parts:
- added D1, D10, D11, D12, D13, D14, D15, D16, D2, D3, D4, D5, D6, D7, D8, D9: LED, LED_SMD:LED_0603_1608Metric_Pad1.05x0.95mm_HandSolder, symbol Device:LED
- added J3, J4: Conn_01x08, Connector_PinHeader_2.54mm:PinHeader_1x08_P2.54mm_Vertical, symbol Connector_Generic:Conn_01x08
- added U1, U2: 40374, Package_DIP:DIP-20_W7.62mm_Socket_LongPads, symbol 4xxx_IEEE:40374
- added U3, U4: 40245, Package_DIP:DIP-20_W7.62mm_Socket_LongPads, symbol 4xxx_IEEE:40245
Connections:
- new net +5V: U1.20 (Vdd), U2.20 (Vdd), U3.1 (Dir), U3.20 (Vdd), U4.20 (Vdd)
- new net BUS1: U1.18, U4.9
- new net BUS10: U2.3, U3.15
- new net BUS11: U2.4, U3.16
- new net BUS12: U2.17, U4.4
- new net BUS13: U2.7, U3.17
- new net BUS14: U2.14, U4.3
- new net BUS15: U2.8, U3.18
- new net BUS16: U2.13, U4.2
- new net BUS2: U1.3, U3.11
- new net BUS3: U1.4, U3.12
- new net BUS4: U1.17, U4.8
- new net BUS5: U1.7, U3.13
- new net BUS6: U1.14, U4.7
- new net BUS7: U1.8, U3.14
- new net BUS8: U1.13, U4.6
- new net BUS9: U2.18, U4.5
- new net GND: D1.1 (K), D10.1 (K), D11.1 (K), D12.1 (K), D13.1 (K), D14.1 (K), D15.1 (K), D16.1 (K), D2.1 (K), D3.1 (K), D4.1 (K), D5.1 (K), D6.1 (K), D7.1 (K), D8.1 (K), D9.1 (K), U1.1 (~{E}), U1.10 (Vss), U2.1 (~{E}), U2.10 (Vss), U3.10 (Vss), U4.1 (Dir), U4.10 (Vss)
- new net LOAD: U1.11 (Ck), U2.11 (Ck)
- new net data1: D1.2 (A), J3.1 (Pin_1), U1.19, U4.11
- new net data10: D10.2 (A), J4.2 (Pin_2), U2.2, U3.5
- new net data11: D11.2 (A), J4.3 (Pin_3), U2.5, U3.4
- new net data12: D12.2 (A), J4.4 (Pin_4), U2.16, U4.16
- new net data13: D13.2 (A), J4.5 (Pin_5), U2.6, U3.3
- new net data14: D14.2 (A), J4.6 (Pin_6), U2.15, U4.17
- new net data15: D15.2 (A), J4.7 (Pin_7), U2.9, U3.2
- new net data16: D16.2 (A), J4.8 (Pin_8), U2.12, U4.18
- new net data2: D2.2 (A), J3.2 (Pin_2), U1.2, U3.9
- new net data3: D3.2 (A), J3.3 (Pin_3), U1.5, U3.8
- new net data4: D4.2 (A), J3.4 (Pin_4), U1.16, U4.12
- new net data5: D5.2 (A), J3.5 (Pin_5), U1.6, U3.7
- new net data6: D6.2 (A), J3.6 (Pin_6), U1.15, U4.13
- new net data7: D7.2 (A), J3.7 (Pin_7), U1.9, U3.6
- new net data8: D8.2 (A), J3.8 (Pin_8), U1.12, U4.14
- new net data9: D9.2 (A), J4.1 (Pin_1), U2.19, U4.15
- new net ~{ENABLE}: U3.19 (~{G}), U4.19 (~{G})
