File: 16bit_computer.kicad_pcb (KiCad board)
At the start: 2 copper layers, 61 x 157.5 mm, 24 parts, among them J1 Conn_01x03, J2 Conn_01x16_Male, U1 40374, U2 40374, U3 40245, U4 40245, U5 7408

Commit message: register finished?
Parts:
- added D17: LED, LED_SMD:LED_0603_1608Metric_Pad1.05x0.95mm_HandSolder, F.Cu at (118.1, 77.5)
- added D18: LED, LED_SMD:LED_0603_1608Metric_Pad1.05x0.95mm_HandSolder, F.Cu at (118.1, 80.0)
- added D19: LED, LED_SMD:LED_0603_1608Metric_Pad1.05x0.95mm_HandSolder, F.Cu at (118.1, 82.5)
- added D20: LED, LED_SMD:LED_0603_1608Metric_Pad1.05x0.95mm_HandSolder, F.Cu at (118.1, 85.1)
- added D21: LED, LED_SMD:LED_0603_1608Metric_Pad1.05x0.95mm_HandSolder, F.Cu at (118.1, 87.6)
- added D22: LED, LED_SMD:LED_0603_1608Metric_Pad1.05x0.95mm_HandSolder, F.Cu at (118.1, 90.2)
- added D23: LED, LED_SMD:LED_0603_1608Metric_Pad1.05x0.95mm_HandSolder, F.Cu at (118.1, 92.7)
- added D24: LED, LED_SMD:LED_0603_1608Metric_Pad1.05x0.95mm_HandSolder, F.Cu at (118.1, 95.2)
- added D25: LED, LED_SMD:LED_0603_1608Metric_Pad1.05x0.95mm_HandSolder, F.Cu at (118.1, 106.7)
- added D26: LED, LED_SMD:LED_0603_1608Metric_Pad1.05x0.95mm_HandSolder, F.Cu at (118.1, 109.2)
- added D27: LED, LED_SMD:LED_0603_1608Metric_Pad1.05x0.95mm_HandSolder, F.Cu at (118.1, 111.8)
- added D28: LED, LED_SMD:LED_0603_1608Metric_Pad1.05x0.95mm_HandSolder, F.Cu at (118.1, 114.3)
- added D29: LED, LED_SMD:LED_0603_1608Metric_Pad1.05x0.95mm_HandSolder, F.Cu at (118.1, 116.8)
- added D30: LED, LED_SMD:LED_0603_1608Metric_Pad1.05x0.95mm_HandSolder, F.Cu at (118.1, 119.4)
- added D31: LED, LED_SMD:LED_0603_1608Metric_Pad1.05x0.95mm_HandSolder, F.Cu at (118.1, 121.9)
- added D32: LED, LED_SMD:LED_0603_1608Metric_Pad1.05x0.95mm_HandSolder, F.Cu at (118.1, 124.5)
- added D33: LED, LED_SMD:LED_0603_1608Metric_Pad1.05x0.95mm_HandSolder, F.Cu at (170.8, 77.5)
- added D34: LED, LED_SMD:LED_0603_1608Metric_Pad1.05x0.95mm_HandSolder, F.Cu at (170.8, 80.0)
- added D35: LED, LED_SMD:LED_0603_1608Metric_Pad1.05x0.95mm_HandSolder, F.Cu at (170.8, 82.5)
- added D36: LED, LED_SMD:LED_0603_1608Metric_Pad1.05x0.95mm_HandSolder, F.Cu at (170.8, 85.1)
- added D37: LED, LED_SMD:LED_0603_1608Metric_Pad1.05x0.95mm_HandSolder, F.Cu at (170.8, 87.6)
- added D38: LED, LED_SMD:LED_0603_1608Metric_Pad1.05x0.95mm_HandSolder, F.Cu at (170.8, 90.2)
- added D39: LED, LED_SMD:LED_0603_1608Metric_Pad1.05x0.95mm_HandSolder, F.Cu at (170.8, 92.7)
- added D40: LED, LED_SMD:LED_0603_1608Metric_Pad1.05x0.95mm_HandSolder, F.Cu at (170.8, 95.2)
- added D41: LED, LED_SMD:LED_0603_1608Metric_Pad1.05x0.95mm_HandSolder, F.Cu at (170.8, 106.7)
- added D42: LED, LED_SMD:LED_0603_1608Metric_Pad1.05x0.95mm_HandSolder, F.Cu at (170.8, 109.2)
- added D43: LED, LED_SMD:LED_0603_1608Metric_Pad1.05x0.95mm_HandSolder, F.Cu at (170.8, 111.8)
- added D44: LED, LED_SMD:LED_0603_1608Metric_Pad1.05x0.95mm_HandSolder, F.Cu at (170.8, 114.3)
- added D45: LED, LED_SMD:LED_0603_1608Metric_Pad1.05x0.95mm_HandSolder, F.Cu at (170.8, 116.8)
- added D46: LED, LED_SMD:LED_0603_1608Metric_Pad1.05x0.95mm_HandSolder, F.Cu at (170.8, 119.4)
- added D47: LED, LED_SMD:LED_0603_1608Metric_Pad1.05x0.95mm_HandSolder, F.Cu at (170.8, 121.9)
- added D48: LED, LED_SMD:LED_0603_1608Metric_Pad1.05x0.95mm_HandSolder, F.Cu at (170.8, 124.5)
- added D49: LED, LED_SMD:LED_0603_1608Metric_Pad1.05x0.95mm_HandSolder, F.Cu at (222.9, 77.5)
- added D50: LED, LED_SMD:LED_0603_1608Metric_Pad1.05x0.95mm_HandSolder, F.Cu at (222.9, 80.0)
- added D51: LED, LED_SMD:LED_0603_1608Metric_Pad1.05x0.95mm_HandSolder, F.Cu at (222.9, 82.5)
- added D52: LED, LED_SMD:LED_0603_1608Metric_Pad1.05x0.95mm_HandSolder, F.Cu at (222.9, 85.1)
- added D53: LED, LED_SMD:LED_0603_1608Metric_Pad1.05x0.95mm_HandSolder, F.Cu at (222.9, 87.6)
- added D54: LED, LED_SMD:LED_0603_1608Metric_Pad1.05x0.95mm_HandSolder, F.Cu at (222.9, 90.2)
- added D55: LED, LED_SMD:LED_0603_1608Metric_Pad1.05x0.95mm_HandSolder, F.Cu at (222.9, 92.7)
- added D56: LED, LED_SMD:LED_0603_1608Metric_Pad1.05x0.95mm_HandSolder, F.Cu at (222.9, 95.2)
- added D57: LED, LED_SMD:LED_0603_1608Metric_Pad1.05x0.95mm_HandSolder, F.Cu at (222.9, 106.7)
- added D58: LED, LED_SMD:LED_0603_1608Metric_Pad1.05x0.95mm_HandSolder, F.Cu at (222.9, 109.2)
- added D59: LED, LED_SMD:LED_0603_1608Metric_Pad1.05x0.95mm_HandSolder, F.Cu at (222.9, 111.8)
- added D60: LED, LED_SMD:LED_0603_1608Metric_Pad1.05x0.95mm_HandSolder, F.Cu at (222.9, 114.3)
- added D61: LED, LED_SMD:LED_0603_1608Metric_Pad1.05x0.95mm_HandSolder, F.Cu at (222.9, 116.8)
- added D62: LED, LED_SMD:LED_0603_1608Metric_Pad1.05x0.95mm_HandSolder, F.Cu at (222.9, 119.4)
- added D63: LED, LED_SMD:LED_0603_1608Metric_Pad1.05x0.95mm_HandSolder, F.Cu at (222.9, 121.9)
- added D64: LED, LED_SMD:LED_0603_1608Metric_Pad1.05x0.95mm_HandSolder, F.Cu at (222.9, 124.5)
- added J10: Conn_01x08, Connector_PinHeader_2.54mm:PinHeader_1x08_P2.54mm_Vertical, F.Cu at (165.7, 106.7)
- added J11: Conn_01x08, Connector_PinHeader_2.54mm:PinHeader_1x08_P2.54mm_Vertical, F.Cu at (217.8, 77.5)
- added J12: Conn_01x08, Connector_PinHeader_2.54mm:PinHeader_1x08_P2.54mm_Vertical, F.Cu at (217.8, 106.7)
- added J3: Conn_01x08, Connector_PinHeader_2.54mm:PinHeader_1x08_P2.54mm_Vertical, F.Cu at (61.0, 77.5)
- added J4: Conn_01x08, Connector_PinHeader_2.54mm:PinHeader_1x08_P2.54mm_Vertical, F.Cu at (61.0, 106.7)
- added J5: Conn_01x08, Connector_PinHeader_2.54mm:PinHeader_1x08_P2.54mm_Vertical, F.Cu at (113.0, 77.5)
- added J6: Conn_01x08, Connector_PinHeader_2.54mm:PinHeader_1x08_P2.54mm_Vertical, F.Cu at (113.0, 106.7)
- added J7: Conn_01x16, Connector_PinHeader_2.54mm:PinHeader_1x16_P2.54mm_Vertical, F.Cu at (228.6, 90.2)
- added J8: Conn_01x16, Connector_PinHeader_2.54mm:PinHeader_1x16_P2.54mm_Vertical, F.Cu at (14.6, 90.2)
- added J9: Conn_01x08, Connector_PinHeader_2.54mm:PinHeader_1x08_P2.54mm_Vertical, F.Cu at (165.7, 77.5)
- added REG2: Conn_01x02, Connector_PinHeader_2.54mm:PinHeader_1x02_P2.54mm_Vertical, F.Cu at (88.9, 191.8)
- added REG3: Conn_01x02, Connector_PinHeader_2.54mm:PinHeader_1x02_P2.54mm_Vertical, F.Cu at (141.6, 191.8)
- added REG4: Conn_01x02, Connector_PinHeader_2.54mm:PinHeader_1x02_P2.54mm_Vertical, F.Cu at (193.7, 191.8)
- added U10: 40374, Package_DIP:DIP-20_W7.62mm_Socket_LongPads, F.Cu at (139.7, 74.9)
- added U11: 40374, Package_DIP:DIP-20_W7.62mm_Socket_LongPads, F.Cu at (139.7, 104.1)
- added U12: 40245, Package_DIP:DIP-20_W7.62mm_Socket_LongPads, F.Cu at (139.7, 162.6)
- added U13: 40245, Package_DIP:DIP-20_W7.62mm_Socket_LongPads, F.Cu at (139.7, 133.3)
- added U14: 40374, Package_DIP:DIP-20_W7.62mm_Socket_LongPads, F.Cu at (191.8, 74.9)
- added U15: 40374, Package_DIP:DIP-20_W7.62mm_Socket_LongPads, F.Cu at (191.8, 104.1)
- added U16: 40245, Package_DIP:DIP-20_W7.62mm_Socket_LongPads, F.Cu at (191.8, 162.6)
- added U17: 40245, Package_DIP:DIP-20_W7.62mm_Socket_LongPads, F.Cu at (191.8, 133.4)
- added U6: 40374, Package_DIP:DIP-20_W7.62mm_Socket_LongPads, F.Cu at (87.0, 74.9)
- added U7: 40374, Package_DIP:DIP-20_W7.62mm_Socket_LongPads, F.Cu at (87.0, 104.1)
- added U8: 40245, Package_DIP:DIP-20_W7.62mm_Socket_LongPads, F.Cu at (87.0, 162.6)
- added U9: 40245, Package_DIP:DIP-20_W7.62mm_Socket_LongPads, F.Cu at (87.0, 133.3)
- D1, D10, D11, D12, D13, D14, D15, D16, D2, D3, D4, D5, D6, D7, D8, D9: footprint Diode_SMD:D_0603_1608Metric_Pad1.05x0.95mm_HandSolder_BETTER -> LED_SMD:LED_0603_1608Metric_Pad1.05x0.95mm_HandSolder
- moved D1 4.44 mm to (66.0, 77.5)
- moved D10 4.44 mm to (66.0, 109.2)
- moved D11 4.44 mm to (66.0, 111.8)
- moved D12 4.44 mm to (66.0, 114.3)
- moved D13 4.44 mm to (66.0, 116.8)
- moved D14 4.44 mm to (66.0, 119.4)
- moved D15 4.44 mm to (66.0, 121.9)
- moved D16 4.44 mm to (66.0, 124.5)
- moved D2 4.44 mm to (66.0, 80.0)
- moved D3 4.44 mm to (66.0, 82.5)
- moved D4 4.44 mm to (66.0, 85.1)
- moved D5 4.44 mm to (66.0, 87.6)
- moved D6 4.44 mm to (66.0, 90.2)
- moved D7 4.44 mm to (66.0, 92.7)
- moved D8 4.44 mm to (66.0, 95.2)
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- renumbered JA1 to REG1
Connections:
- net /1 renamed /BUS1
- net /10 renamed /BUS10
- net /11 renamed /BUS11
- net /12 renamed /BUS12
- net /13 renamed /BUS13
- net /14 renamed /BUS14
- net /15 renamed /BUS15
- net /16 renamed /BUS16
- net /2 renamed /BUS2
- net /3 renamed /BUS3
- net /4 renamed /BUS4
- net /5 renamed /BUS5
- net /6 renamed /BUS6
- net /7 renamed /BUS7
- net /8 renamed /BUS8
- net /9 renamed /BUS9
- net LOAD_A renamed /Register1/LOAD
- net Net-(D1-Pad2) renamed /Register1/data1
- net Net-(D10-Pad2) renamed /Register1/data10
- net Net-(D11-Pad2) renamed /Register1/data11
- net Net-(D12-Pad2) renamed /Register1/data12
- net Net-(D13-Pad2) renamed /Register1/data13
- net Net-(D14-Pad2) renamed /Register1/data14
- net Net-(D15-Pad2) renamed /Register1/data15
- net Net-(D16-Pad2) renamed /Register1/data16
- net Net-(D2-Pad2) renamed /Register1/data2
- net Net-(D3-Pad2) renamed /Register1/data3
- net Net-(D4-Pad2) renamed /Register1/data4
- net Net-(D5-Pad2) renamed /Register1/data5
- net Net-(D6-Pad2) renamed /Register1/data6
- net Net-(D7-Pad2) renamed /Register1/data7
- net Net-(D8-Pad2) renamed /Register1/data8
- net Net-(D9-Pad2) renamed /Register1/data9
- net ~{EN_A} renamed /Register1/~{ENABLE}
- REG1 pad 2: LD_A -> Net-(REG1-Pad2)
- U5 pad 1: unconnected-(U5-Pad1) -> Net-(REG3-Pad2)
- U5 pad 10: unconnected-(U5-Pad10) -> Net-(REG4-Pad2)
- U5 pad 11: unconnected-(U5-Pad11) -> /Register2/LOAD
- U5 pad 12: unconnected-(U5-Pad12) -> CLK
- U5 pad 13: unconnected-(U5-Pad13) -> Net-(REG2-Pad2)
- U5 pad 2: unconnected-(U5-Pad2) -> CLK
- U5 pad 3: unconnected-(U5-Pad3) -> /Register3/LOAD
- U5 pad 4: CLK -> Net-(REG1-Pad2)
- U5 pad 5: LD_A -> CLK
- U5 pad 8: unconnected-(U5-Pad8) -> /Register4/LOAD
- U5 pad 9: unconnected-(U5-Pad9) -> CLK
Routing:
- net /BUS14: track 308.3 -> 1224.6 mm, vias 3 -> 9
- net /BUS16: track 262.2 -> 1043.8 mm, vias 3 -> 9
- net GND: track 297.1 -> 1055.4 mm, vias 5 -> 21
- net /BUS12: track 244.6 -> 966.0 mm, vias 3 -> 9
- net /BUS9: track 238.7 -> 936.9 mm, vias 3 -> 9
- net /BUS8: track 232.9 -> 912.8 mm, vias 3 -> 9
- net /BUS6: track 227.1 -> 888.5 mm, vias 3 -> 9
- net /BUS4: track 221.2 -> 860.3 mm, vias 3 -> 9
- net /BUS1: track 217.4 -> 825.0 mm, vias 3 -> 9
- net /BUS15: track 184.6 -> 731.5 mm, vias 3 -> 12
- net /BUS13: track 185.3 -> 730.6 mm, vias 4 -> 13
- net /BUS11: track 185.3 -> 726.5 mm, vias 4 -> 13
- net /BUS10: track 182.8 -> 715.5 mm, vias 4 -> 13
- net /BUS7: track 182.8 -> 712.6 mm, vias 4 -> 13
- net /BUS5: track 182.8 -> 708.2 mm, vias 4 -> 13
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Other:
- board size 61 x 157.5 mm -> 219.1 x 157.5 mm
- board text added: "1"
- board text added: "10"
- board text added: "11"
- board text added: "12"
- board text added: "13"
- board text added: "14"
- board text added: "15"
- board text added: "16"
- board text added: "2"
- board text added: "3"
- board text added: "4"
- board text added: "5"
- board text added: "6"
- board text added: "7"
- board text added: "8"
- board text added: "9"

Commit message: final v0.3
Routing:
- net GND: track 1055.4 -> 984.5 mm, vias 21 -> 18
- net /BUS16: track 1043.8 -> 1022.8 mm
- net /BUS1: track 825.0 -> 834.0 mm
- net /BUS15: track 731.5 -> 725.5 mm
- net /Register4/data3: track 103.8 -> 101.6 mm
- net /Register3/data3: track 103.8 -> 101.6 mm
- net /Register2/data3: track 103.8 -> 101.6 mm
- net /Register1/data3: track 103.8 -> 101.6 mm
- net +5V: track 645.5 -> 643.6 mm
- net /BUS10: track 715.5 -> 714.8 mm
- net Net-(REG4-Pad2): track 130.1 -> 129.5 mm
